Commit message: fixed inertia

File: calypso_sim/urdf/auv.urdf.xacro (robot description, xacro)
@@ -23,10 +23,4 @@
     <!-- <xacro:property name="x" default="0"/>
     <xacro:property name="y" default="0"/> -->
-    <xacro:property name="x" default="-0.26"/>
-    <xacro:property name="y" default="0.43"/>
-    <xacro:property name="z" default="0"/>
-    <xacro:property name="r" default="1.57"/>
-    <xacro:property name="p" default="0"/>
-    <xacro:property name="Y" default="0"/>
     <xacro:base_link xyz="0 0 0" rpy="0 1.57 0"></xacro:base_link>
     <!--

File: calypso_sim/urdf/chasis.urdf.xacro (robot description, xacro)
@@ -21,6 +21,6 @@
     </inertial> -->
     <inertial>
-      <mass value="38.00000000"/>
-      <inertia ixx="1029167.62033618" ixy="-0.00000959" ixz="-0.00004980" iyy="1512698.34325725" iyz="1440.15048769" izz="708288.26651739"/>
+      <mass value="5"/>
+      <inertia ixx="0" ixy="0" ixz="0" iyy="0" iyz="0" izz="0"/>
     </inertial>
   </link>

Commit message: integrated pid and fixed heave pid

File: calypso_sim/urdf/auv.urdf.xacro (robot description, xacro)
@@ -1,9 +1,10 @@
 <?xml version="1.0"?>
 <robot xmlns:xacro="http://www.ros.org/wiki/xacro" name="auv">
-    <xacro:include filename="$(find calypso_sim)/urdf/camera2d.urdf.xacro"/>
-    <xacro:include filename="$(find calypso_sim)/urdf/camera_depth.urdf.xacro"/>
+    <!-- <xacro:include filename="$(find calypso_sim)/urdf/camera2d.urdf.xacro"/> -->
+    <!-- <xacro:include filename="$(find calypso_sim)/urdf/camera_depth.urdf.xacro"/> -->
     <xacro:include filename="$(find calypso_sim)/urdf/imu.urdf.xacro"/>
     <xacro:include filename="$(find calypso_sim)/urdf/thrusters.urdf.xacro"/>
     <xacro:include filename="$(find calypso_sim)/urdf/chasis.urdf.xacro"/>
+    <xacro:include filename="$(find calypso_sim)/urdf/dvl_snippets.urdf.xacro"/>
     <material name="red">
         <color rgba="1 0 0 1"/>
@@ -50,6 +51,8 @@
     <xacro:thruster_CCW id="8" parent="base_link" xyz="-0.45 0.2 0" rpy="0 1.57 0.785398" axis="0 0 -1">
     </xacro:thruster_CCW>
-    <xacro:imu id="1" parent="base_link" xyz="0 0 0.15" rpy="0 0 -1.57">
-    </xacro:imu>
+    <xacro:default_dvl namespace="calypso_sim" parent_link="base_link">
+      <origin xyz="0 0 -0.18" rpy="0 0 0"/>
+    </xacro:default_dvl>
+    <xacro:imu id="1" parent="base_link" xyz="0 0 0" rpy="0 0 0"></xacro:imu>
     <gazebo>
       <plugin name="gazebo_ros_control" filename="libgazebo_ros_control.so">
@@ -58,23 +61,23 @@
       </plugin>
     </gazebo>
-  <gazebo>
-    <plugin name="freebuoyancy_gazebo" filename="libfreebuoyancy_gazebo.so">
-      <descriptionParam>robot_description</descriptionParam>
-      <alwaysOn>true</alwaysOn>
-      <surface>0 0 40</surface>
-      <updateRate>.001</updateRate>
-      <link name='base_link'>
-        <buoyancy>
-          <compensation>0.0</compensation>
-          <origin xyz="0 0 0"/>
-        </buoyancy>
-      </link>
-    </plugin>
-  </gazebo>
+    <gazebo>
+      <plugin name="freebuoyancy_gazebo" filename="libfreebuoyancy_gazebo.so">
+        <descriptionParam>/robot_description</descriptionParam>
+        <alwaysOn>true</alwaysOn>
+        <surface>0 0 40</surface>
+        <updateRate>.001</updateRate>
+        <link name='base_link'>
+          <buoyancy>
+            <compensation>0.0</compensation>
+            <origin xyz="0 0 0"/>
+          </buoyancy>
+        </link>
+      </plugin>
+    </gazebo>
   <!-- <gazebo>
     <plugin name="BuoyancyPlugin" filename="libBuoyancyPlugin.so">
-    <fluid_density>1000</fluid_density>
+    <fluid_density>1200</fluid_density>
     <link name="base_link">
-      <volume>0.03</volume>
+      <volume>240</volume>
       <center_of_volume>0 0 0</center_of_volume>
     </link>

File: calypso_sim/urdf/chasis.urdf.xacro (robot description, xacro)
@@ -17,9 +17,9 @@
     </collision>
     <!-- <inertial>
-      <mass value="37"/>
+      <mass value="40"/>
       <inertia ixx="1002084.26190628" ixy="-0.00000934" ixz="-0.00004849" iyy="1472890.49211890" iyz="1402.25179064" izz="689649.10160904"/>
     </inertial> -->
     <inertial>
-      <mass value="5"/>
+      <mass value="42.775"/>
       <inertia ixx="0" ixy="0" ixz="0" iyy="0" iyz="0" izz="0"/>
     </inertial>

File: calypso_sim/urdf/imu.urdf.xacro (robot description, xacro)
@@ -35,6 +35,10 @@
                 <alwaysOn>true</alwaysOn>
                 <gaussianNoise>0</gaussianNoise>
+                <updateRate>10.0</updateRate>
             </plugin>
         </gazebo>
     </xacro:macro>
+    <!-- <link name="base_link">
+    </link>
+    <xacro:imu id="1" parent="base_link" xyz="0 0 0" rpy="0 0 0"></xacro:imu> -->
 </robot>

Commit message: fixed both pids

File: calypso_sim/urdf/auv.urdf.xacro (robot description, xacro)
@@ -1,5 +1,5 @@
 <?xml version="1.0"?>
 <robot xmlns:xacro="http://www.ros.org/wiki/xacro" name="auv">
-    <!-- <xacro:include filename="$(find calypso_sim)/urdf/camera2d.urdf.xacro"/> -->
+    <xacro:include filename="$(find calypso_sim)/urdf/camera2d.urdf.xacro"/>
     <!-- <xacro:include filename="$(find calypso_sim)/urdf/camera_depth.urdf.xacro"/> -->
     <xacro:include filename="$(find calypso_sim)/urdf/imu.urdf.xacro"/>
@@ -24,5 +24,5 @@
     <!-- <xacro:property name="x" default="0"/>
     <xacro:property name="y" default="0"/> -->
-    <xacro:base_link xyz="0 0 0" rpy="0 1.57 0"></xacro:base_link>
+    <xacro:base_link xyz="0 0 0" rpy="0 1.57 0 "></xacro:base_link>
     <!--
 // 2:right upper 1->2
@@ -55,4 +55,5 @@
     </xacro:default_dvl>
     <xacro:imu id="1" parent="base_link" xyz="0 0 0" rpy="0 0 0"></xacro:imu>
+    <xacro:camera2d id="1" parent="base_link" xyz="0 0.3 0" rpy="0 0 0"></xacro:camera2d>
     <gazebo>
       <plugin name="gazebo_ros_control" filename="libgazebo_ros_control.so">

File: calypso_sim/urdf/camera2d.urdf.xacro (robot description, xacro)
@@ -2,4 +2,5 @@
 <robot xmlns:xacro="http://www.ros.org/wiki/xacro" name="camera">
 <!-- this is for the 2d camera in the bottom -->
+  <xacro:macro name="camera2d" params="id parent xyz rpy">
     <link name="camera_bottom">
       <visual>
@@ -9,19 +10,20 @@
         <material name="red"/>
       </visual>
-      <collision>
+      <!-- <collision>
         <geometry>
           <box size="0.05 0.05 0.05"/>
         </geometry>
-      </collision>
-      <inertial>
-        <mass value="1.5"/>
+      </collision> -->
+      <!-- <inertial>
+        <mass value="0.05"/>
         <origin xyz="0.0 0.0 0.0" rpy="0 0 0"/>
         <inertia ixx="0.0" ixy="0.0" ixz="0.0" iyy="0.0" iyz="0.0" izz="0.0"/>
-      </inertial>
+      </inertial> -->
     </link>
+    <link name="camera_link_optical_bottom"></link>
     <joint name="base_link_to_camera_bottom_joint" type="fixed">
-      <parent link="base_link"/>
+      <parent link="${parent}"/>
       <child link="camera_bottom"/>
-      <origin xyz="0 0 -0.19" rpy="1.57 1.57 0"/>
+      <origin xyz="${xyz}" rpy="${rpy}"/>
     </joint>
     <joint name="camera_optical_joint_bottom" type="fixed">
@@ -30,5 +32,4 @@
       <origin xyz="0 0 0" rpy="${-pi/2} 0 ${-pi/2}"/>
     </joint>
-    <link name="camera_link_optical_bottom"></link>
     <gazebo reference="camera_bottom">
       <material>Gazebo/Red</material>
@@ -56,3 +57,4 @@
       </sensor>
     </gazebo>
+  </xacro:macro>
 </robot>

File: calypso_sim/urdf/camera_depth.urdf.xacro (robot description, xacro)
@@ -62,10 +62,10 @@
           <alwaysOn>true</alwaysOn>
           <!-- <updateRate>0.0</updateRate> -->
-          <cameraName>calypso_sim/camera_front</cameraName>
-          <imageTopicName>/yash_cam/image_raw</imageTopicName>
+          <cameraName>calypso_sim/depth_camera</cameraName>
+          <imageTopicName>image</imageTopicName>
           <!-- <cameraInfoTopicName>camera_info</cameraInfoTopicName> -->
-          <depthImageTopicName>image_raw</depthImageTopicName>
+          <depthImageTopicName>depth_image</depthImageTopicName>
           <depthImageCameraInfoTopicName>camera_info</depthImageCameraInfoTopicName>
-          <pointCloudTopicName>points</pointCloudTopicName>
+          <pointCloudTopicName>3dpoints</pointCloudTopicName>
           <!-- <frameName>camera_link</frameName> -->
           <pointCloudCutoff>0.5</pointCloudCutoff>

File: calypso_sim/urdf/imu.urdf.xacro (robot description, xacro)
@@ -29,5 +29,5 @@
                 <topicName>/calypso_sim/imu/data</topicName>
                 <serviceName>/calypso_sim/imu/service</serviceName>
-                <bodyName>base_link</bodyName>
+                <bodyName>imu_${id}</bodyName>
                 <gaussianNoise>0</gaussianNoise>
                 <rpyOffsets>0 0 0</rpyOffsets>

Commit message: fixed visualization node and started pid tuning

File: calypso_sim/urdf/auv.urdf.xacro (robot description, xacro)
@@ -1,6 +1,6 @@
 <?xml version="1.0"?>
 <robot xmlns:xacro="http://www.ros.org/wiki/xacro" name="auv">
-    <xacro:include filename="$(find calypso_sim)/urdf/camera2d.urdf.xacro"/>
-    <!-- <xacro:include filename="$(find calypso_sim)/urdf/camera_depth.urdf.xacro"/> -->
+    <!-- <xacro:include filename="$(find calypso_sim)/urdf/camera2d.urdf.xacro"/> -->
+    <xacro:include filename="$(find calypso_sim)/urdf/camera_depth.urdf.xacro"/>
     <xacro:include filename="$(find calypso_sim)/urdf/imu.urdf.xacro"/>
     <xacro:include filename="$(find calypso_sim)/urdf/thrusters.urdf.xacro"/>
@@ -55,5 +55,5 @@
     </xacro:default_dvl>
     <xacro:imu id="1" parent="base_link" xyz="0 0 0" rpy="0 0 0"></xacro:imu>
-    <xacro:camera2d id="1" parent="base_link" xyz="0 0.3 0" rpy="0 0 0"></xacro:camera2d>
+    <xacro:depth_cam id="1" parent="base_link" xyz="0.3 0 0" rpy="0 0 0"></xacro:depth_cam>
     <gazebo>
       <plugin name="gazebo_ros_control" filename="libgazebo_ros_control.so">

File: calypso_sim/urdf/camera2d.urdf.xacro (robot description, xacro)
@@ -1,7 +1,7 @@
 <?xml version="1.0"?>
 <robot xmlns:xacro="http://www.ros.org/wiki/xacro" name="camera">
-<!-- this is for the 2d camera in the bottom -->
+<!-- this is for the 2d camera in the front -->
   <xacro:macro name="camera2d" params="id parent xyz rpy">
-    <link name="camera_bottom">
+    <link name="camera_front">
       <visual>
         <geometry>
@@ -21,16 +21,16 @@
       </inertial> -->
     </link>
-    <link name="camera_link_optical_bottom"></link>
-    <joint name="base_link_to_camera_bottom_joint" type="fixed">
+    <link name="camera_link_optical_front"></link>
+    <joint name="base_link_to_camera_front_joint" type="fixed">
       <parent link="${parent}"/>
-      <child link="camera_bottom"/>
+      <child link="camera_front"/>
       <origin xyz="${xyz}" rpy="${rpy}"/>
     </joint>
-    <joint name="camera_optical_joint_bottom" type="fixed">
-      <parent link="camera_bottom"/>
-      <child link="camera_link_optical_bottom"/>
+    <joint name="camera_optical_joint_front" type="fixed">
+      <parent link="camera_front"/>
+      <child link="camera_link_optical_front"/>
       <origin xyz="0 0 0" rpy="${-pi/2} 0 ${-pi/2}"/>
     </joint>
-    <gazebo reference="camera_bottom">
+    <gazebo reference="camera_front">
       <material>Gazebo/Red</material>
       <sensor name="camera" type="camera">
@@ -51,6 +51,6 @@
         </camera>
         <plugin name="camera_controller" filename="libgazebo_ros_camera.so">
-          <frame_name>camera_link_optical_bottom</frame_name>
-          <cameraName>calypso_sim/camera_bottom</cameraName>
+          <frame_name>camera_link_optical_front</frame_name>
+          <cameraName>calypso_sim/camera_front</cameraName>
           <imageTopicName>image_raw</imageTopicName>
         </plugin>

File: calypso_sim/urdf/camera_depth.urdf.xacro (robot description, xacro)
@@ -1,86 +1,72 @@
 <?xml version="1.0"?>
-<robot xmlns:xacro="http://www.ros.org/wiki/xacro" name="camera">
-<!-- this is for the depth camera in the front -->
-    <link name="camera_front">
+<robot xmlns:xacro="http://www.ros.org/wiki/xacro" id="depth_cam">
+  <xacro:macro name="depth_cam" params="id parent xyz rpy">
+    <joint name="depth_cam_${id}_joint" type="fixed">
+      <origin xyz="${xyz}" rpy="${rpy}"/>
+      <parent link="${parent}"/>
+      <child link="depth_cam_${id}_link"/>
+    </joint>
+    <link name="depth_cam_${id}_link">
+      <collision>
+          <geometry>
+              <box size="0.05 0.05 0.05"/>
+          </geometry>
+      </collision>
       <visual>
-        <geometry>
-          <box size="0.05 0.05 0.05"/>
-        </geometry>
-        <material name="red"/>
+          <geometry>
+              <box size="0.05 0.05 0.05"/>
+          </geometry>
+          <material name="blue"/>
       </visual>
-      <collision>
-        <geometry>
-          <box size="0.05 0.05 0.05"/>
-        </geometry>
-      </collision>
       <inertial>
-        <mass value="1.5"/>
-        <origin xyz="0.0 0.0 0.0" rpy="0 0 0"/>
-        <inertia ixx="0.0" ixy="0.0" ixz="0.0" iyy="0.0" iyz="0.0" izz="0.0"/>
+          <mass value="0.0001" />
+          <origin xyz="0 0 0" rpy="0 0 ${pi}"/>
+          <inertia ixx="0.0" ixy="0" ixz="0" iyy="0.0" iyz="0" izz="0.0" />
       </inertial>
     </link>
-    <joint name="base_link_to_camera_front_joint" type="fixed">
-      <parent link="base_link"/>
-      <child link="camera_front"/>
-      <origin xyz="0.3 0 0" rpy="0 0 0"/>
+    <joint name="camera_optical_joint" type="fixed">
+      <!-- these values have to be these values otherwise the gazebo camera
+          image won't be aligned properly with the frame it is supposedly
+          originating from -->
+      <origin xyz="0 0 0" rpy="${-pi/2} 0 ${-pi/2}"/>
+      <parent link="depth_cam_${id}_link"/>
+      <child link="depth_cam_${id}_link_optical"/>
     </joint>
-    <joint name="camera_optical_joint_front" type="fixed">
-      <parent link="camera_front"/>
-      <child link="camera_link_optical_front"/>
-      <origin xyz="0 0 0" rpy="${-pi/2} 0 ${-pi/2}"/>
-    </joint>
-    <link name="camera_link_optical_front"></link>
-    <gazebo reference="camera_front">
-      <material>Gazebo/Red</material>
-      <sensor name="camera" type="depth">
-        <pose> 0 0 0 0 0 0 </pose>
+    <link name="depth_cam_${id}_link_optical">
+    </link>
+    <gazebo reference="depth_cam_${id}_link">
+      <sensor type="depth" name="depth_camera_${id}">
+        <origin xyz="0 0 0" rpy="0 0 0"/>
         <visualize>true</visualize>
-        <update_rate>10</update_rate>
-        <camera>
-          <horizontal_fov>1.089</horizontal_fov>
-          <image>
-            <format>B8G8R8</format>
-            <width>640</width>
-            <height>480</height>
-          </image>
-          <clip>
-            <near>0.05</near>
-            <far>8.0</far>
-          </clip>
-        </camera>
-        <plugin name="camera_plugin" filename="libgazebo_ros_openni_kinect.so">
-          <frame_name>camera_link_optical_front</frame_name>
-          <!-- <min_depth>0.1</min_depth>
-          <max_depth>100.0</max_depth> -->
-          <!-- <cameraName>calypso_sim/camera_front</cameraName>
-          <imageTopicName>image_raw</imageTopicName>
-          <depthImageTopicName>/calypso_sim/camera_front/image_raw</depthImageTopicName>
-          <pointCloudTopicName>/calypso_sim/camera_front/points</pointCloudTopicName>
-          <frameName>camera_link</frameName>
-          <pointCloudCutoff>0.5</pointCloudCutoff>
-          <pointCloudCutoffMax>3.0</pointCloudCutoffMax> -->
-          <alwaysOn>true</alwaysOn>
-          <!-- <updateRate>0.0</updateRate> -->
-          <cameraName>calypso_sim/depth_camera</cameraName>
-          <imageTopicName>image</imageTopicName>
-          <!-- <cameraInfoTopicName>camera_info</cameraInfoTopicName> -->
-          <depthImageTopicName>depth_image</depthImageTopicName>
-          <depthImageCameraInfoTopicName>camera_info</depthImageCameraInfoTopicName>
-          <pointCloudTopicName>3dpoints</pointCloudTopicName>
-          <!-- <frameName>camera_link</frameName> -->
-          <pointCloudCutoff>0.5</pointCloudCutoff>
-          <pointCloudCutoffMax>3.0</pointCloudCutoffMax>
-          <!-- <distortionK1>0</distortionK1>
-          <distortionK2>0</distortionK2>
-          <distortionK3>0</distortionK3>
-          <distortionT1>0</distortionT1>
-          <distortionT2>0</distortionT2>
-          <CxPrime>0</CxPrime>
-          <Cx>0</Cx>
-          <Cy>0</Cy>
-          <focalLength>0</focalLength>
-          <hackBaseline>0</hackBaseline> -->
-        </plugin>
+        <update_rate>40</update_rate>
+          <plugin name="depth_camera_${id}_plugin" filename="libgazebo_ros_openni_kinect.so">
+            <baseline>0.2</baseline>
+            <alwaysOn>true</alwaysOn>
+            <!-- Keep this zero, update_rate in the parent <sensor> tag
+              will control the frame rate. -->
+            <updateRate>0.0</updateRate>
+            <cameraName>camera_ir</cameraName>
+            <robotNamespace>/calypso_sim</robotNamespace>
+            <imageTopicName>/camera/depth/image_raw</imageTopicName>
+            <cameraInfoTopicName>/camera/depth/camera_info</cameraInfoTopicName>
+            <depthImageTopicName>/camera/depth/image_raw</depthImageTopicName>
+            <depthImageInfoTopicName>/camera/depth/camera_info</depthImageInfoTopicName>
+            <pointCloudTopicName>/camera/depth/points</pointCloudTopicName>
+            <frameName>depth_cam_${id}_link_optical</frameName>
+            <pointCloudCutoff>0.05</pointCloudCutoff>
+            <distortionK1>0</distortionK1>
+            <distortionK2>0</distortionK2>
+            <distortionK3>0</distortionK3>
+            <distortionT1>0</distortionT1>
+            <distortionT2>0</distortionT2>
+            <CxPrime>0</CxPrime>
+            <Cx>0</Cx>
+            <Cy>0</Cy>
+            <focalLength>0</focalLength>
+            <hackBaseline>0</hackBaseline>
+          </plugin>
       </sensor>
+      <static>true</static>
     </gazebo>
-  </robot>
+  </xacro:macro>
+</robot>

File: calypso_sim/urdf/imu.urdf.xacro (robot description, xacro)
@@ -25,5 +25,5 @@
             </inertial>
         </link>
-=       <gazebo>
+       <gazebo>
             <plugin name="gazebo_ros_imu_${id}_controller" filename="libgazebo_ros_imu.so">
                 <topicName>/calypso_sim/imu/data</topicName>
